File: hardware/kicad/PortaNet/PortaNet.kicad_pcb (KiCad board)
At the start: 2 copper layers, 47.5 x 16.8 mm, 32 parts, among them J1 UART, J2 Molex 0480370001, J3 OLED_PINS, J4 GRPB052VWVN-RC, U1 ESP32-C3, U2 AP2114HA-3.3TRG1, Y1 FL400WFQA1

Commit message: board v2 changes
Parts:
- removed D4: DSS13UTR, Diode_SMD:D_SOD-123F
- removed J4: GRPB052VWVN-RC, Connector_PinHeader_1.27mm:PinHeader_2x05_P1.27mm_Vertical
- removed R2, R3: 0, Resistor_SMD:R_0805_2012Metric
- added C1: 1uF, Capacitor_SMD:C_0603_1608Metric, B.Cu at (150.5, 76.6)
- J1: footprint Connector_PinSocket_2.54mm:PinSocket_1x03_P2.54mm_Vertical -> Connector_PinSocket_2.54mm:PinSocket_1x04_P2.54mm_Vertical
- moved TP4 3.78 mm to (162.6, 64.3)
- moved J3 0.64 mm to (161.5, 67.3)
- moved H1 0.25 mm to (166.2, 71.1)
Connections:
- U1 pad 10: JTAG_TDI -> unconnected-(U1-Pad10)
- U1 pad 12: JTAG_TCK -> unconnected-(U1-Pad12)
- U1 pad 13: JTAG_TDO -> unconnected-(U1-Pad13)
- U1 pad 25: unconnected-(U1-Pad25) -> USB_DN
- U1 pad 26: unconnected-(U1-Pad26) -> USB_DP
- U1 pad 9: JTAG_TMS -> unconnected-(U1-Pad9)
Routing:
- net 5V: track 18.1 -> 38.4 mm
- net GND: track 27.9 -> 44.7 mm, vias 2 -> 4
- net USB_DN: track 7.42 -> 20.1 mm
- net JTAG_TMS: track 12.3 -> 0.00 mm, vias 1 -> 0
- net JTAG_TDI: track 8.98 -> 0.00 mm, vias 1 -> 0
- net 3V3: track 31.3 -> 22.6 mm, vias 7 -> 8
- net USB_DP: track 6.78 -> 15.1 mm, vias 0 -> 2
- net Net-(J1-Pad3): track 17.4 -> 9.68 mm
- net JTAG_TCK: track 7.38 -> 0.00 mm
- net JTAG_TDO: track 6.06 -> 0.00 mm
- net Net-(R1-Pad1): track 3.03 -> 7.37 mm, vias 0 -> 1
- net Net-(J1-Pad2): track 14.2 -> 9.99 mm
- net Net-(D4-Pad2): track 2.79 -> 0.00 mm
- net I2C_SCL: track 13.0 -> 14.1 mm
- net I2C_SDA: track 11.9 -> 12.5 mm
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Other:
- board text added: "3.3V"
- board text added: "5V"
- board text added: "GND"
- board text added: "PortaNet v2.0, A JCM Design"
- board text added: "RX"
- board text added: "TX"
- board text removed: "PortaNet v1.0, A JCM Design"
