File: hardware/kicad/PortaNet/esp32.kicad_sch (KiCad schematic)
At the start: 0 parts

Commit message: update sch
Parts:
- added U?: ESP32-C3, Package_DFN_QFN:QFN-32-1EP_5x5mm_P0.5mm_EP3.7x3.7mm_ThermalVias, symbol JoesSymbols:ESP32-C3
Changed lines of the file:
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@@
 (kicad_sch (version 20211123) (generator eeschema)
   (paper "A4")
+  (symbol (lib_id "JoesSymbols:ESP32-C3") (at 118.11 69.85 0) (unit 1)
+    (in_bom yes) (on_board yes) (fields_autoplaced)
+    (property "Reference" "U?" (id 0) (at 136.6394 118.11 0)
+      (effects (font (size 1.27 1.27)) (justify left))
+    )
+    (property "Value" "ESP32-C3" (id 1) (at 136.6394 120.65 0)
+      (effects (font (size 1.27 1.27)) (justify left))
+    )
+    (property "Footprint" "Package_DFN_QFN:QFN-32-1EP_5x5mm_P0.5mm_EP3.7x3.7mm_ThermalVias" (id 2) (at 83.185 58.42 0)
+      (effects (font (size 1.27 1.27)) hide)
+    )
+    (property "Datasheet" "" (id 3) (at 118.11 69.85 0)
+      (effects (font (size 1.27 1.27)) hide)
+    )
+    (pin "1")
+    (pin "10")
+    (pin "11")
+    (pin "12")
+    (pin "13")
+    (pin "14")
+    (pin "15")
+    (pin "16")
+    (pin "17")
+    (pin "18")
+    (pin "19")
+    (pin "2")
+    (pin "20")
+    (pin "21")
+    (pin "22")
+    (pin "23")
+    (pin "24")
+    (pin "25")
+    (pin "26")
+    (pin "27")
+    (pin "28")
+    (pin "29")
+    (pin "3")
+    (pin "30")
+    (pin "31")
+    (pin "32")
+    (pin "33")
+    (pin "4")
+    (pin "5")
+    (pin "6")
+    (pin "7")
+    (pin "8")
+    (pin "9")
+  )
 )

Commit message: add notes
Connections:
- net 3V3: now reaches U?.11 (VDD3P3_RTC)
- net 3V3: now also U?.17 (VDD3P3_CPU), U?.2 (VDD3P3), U?.3 (VDD3P3), U?.31 (VDDA), U?.32 (VDDA)
- net GND: now reaches U?.33 (GND)
Other:
- moved on the sheet: U?

Commit message: eod commit
Parts:
- added C? (x4): 0.1uF, Capacitor_SMD:C_0603_1608Metric, symbol Device:C_Small
- added C? (x4): 10uF, Capacitor_SMD:C_0603_1608Metric, symbol Device:C_Small
Connections:
- net 3V3: now also C?.1, C?.1, C?.1, C?.1, C?.1, C?.1, C?.1, C?.1
- net GND: now also C?.2, C?.2, C?.2, C?.2, C?.2, C?.2, C?.2, C?.2
Other:
- moved on the sheet: U?

Commit message: eod commit
Parts:
- added J?: UART, Connector_PinSocket_2.54mm:PinSocket_1x03_P2.54mm_Vertical, symbol Connector_Generic:Conn_01x03
- added R?: 10k, Resistor_SMD:R_0805_2012Metric, symbol Device:R_Small_US
Connections:
- net 3V3: now also R?.2
- net GND: now also J?.1 (Pin_1)
- net JTAG_TDI: now reaches U?.10 (MTDI)
- net JTAG_TCK: now reaches U?.12 (MTCK)
- net JTAG_TDO: now reaches U?.13 (MTDO)
- net at U?.27 (U0RXD): now also J?.3 (Pin_3)
- net at U?.28 (U0TXD): now also J?.2 (Pin_2)
- net XTAL_N: now reaches U?.29 (XTAL_N)
- net XTAL_P: now reaches U?.30 (XTAL_P)
- net at U?.7 (CHIP_EN): now also R?.1
- net JTAG_TMS: now reaches U?.9 (MTMS)
- no-connect marks 0 -> 16
Changed lines of the file:
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@@
   (junction (at 114.3 41.275) (diameter 0) (color 0 0 0 0)
   )
+  (no_connect (at 123.825 76.2))
+  (no_connect (at 123.825 73.025))
+  (no_connect (at 123.825 69.85))
+  (no_connect (at 123.825 66.675))
+  (no_connect (at 76.2 88.9))
+  (no_connect (at 76.2 92.075))
+  (no_connect (at 123.825 107.95))
+  (no_connect (at 123.825 104.775))
+  (no_connect (at 123.825 101.6))
+  (no_connect (at 123.825 98.425))
+  (no_connect (at 123.825 95.25))
+  (no_connect (at 123.825 92.075))
+  (no_connect (at 123.825 88.9))
+  (no_connect (at 123.825 85.725))
+  (no_connect (at 123.825 82.55))
+  (no_connect (at 123.825 79.375))
+  (wire (pts (xy 69.215 66.675) (xy 76.2 66.675))
+    (stroke (width 0) (type default) (color 0 0 0 0))
+  )
+  (wire (pts (xy 69.215 69.85) (xy 76.2 69.85))
+    (stroke (width 0) (type default) (color 0 0 0 0))
+  )
   (wire (pts (xy 103.505 40.005) (xy 111.76 40.005))
     (stroke (width 0) (type default) (color 0 0 0 0))
@@
     (stroke (width 0) (type default) (color 0 0 0 0))
   )
+  (wire (pts (xy 46.99 79.375) (xy 46.99 76.2))
+    (stroke (width 0) (type default) (color 0 0 0 0))
+  )
   (wire (pts (xy 114.3 41.275) (xy 116.205 41.275))
     (stroke (width 0) (type default) (color 0 0 0 0))
@@
     (stroke (width 0) (type default) (color 0 0 0 0))
   )
+  (wire (pts (xy 48.26 95.25) (xy 76.2 95.25))
+    (stroke (width 0) (type default) (color 0 0 0 0))
+  )
   (wire (pts (xy 74.295 52.705) (xy 76.2 52.705))
     (stroke (width 0) (type default) (color 0 0 0 0))
@@
     (stroke (width 0) (type default) (color 0 0 0 0))
   )
+  (wire (pts (xy 69.215 73.025) (xy 76.2 73.025))
+    (stroke (width 0) (type default) (color 0 0 0 0))
+  )
   (wire (pts (xy 111.76 36.83) (xy 111.76 40.005))
     (stroke (width 0) (type default) (color 0 0 0 0))
@@
     (stroke (width 0) (type default) (color 0 0 0 0))
   )
+  (wire (pts (xy 46.99 67.945) (xy 46.99 71.12))
+    (stroke (width 0) (type default) (color 0 0 0 0))
+  )
+  (wire (pts (xy 72.39 97.79) (xy 48.26 97.79))
+    (stroke (width 0) (type default) (color 0 0 0 0))
+  )
+  (wire (pts (xy 69.215 82.55) (xy 76.2 82.55))
+    (stroke (width 0) (type default) (color 0 0 0 0))
+  )
+  (wire (pts (xy 76.2 79.375) (xy 46.99 79.375))
+    (stroke (width 0) (type default) (color 0 0 0 0))
+  )
   (wire (pts (xy 126.365 52.705) (xy 128.905 52.705))
     (stroke (width 0) (type default) (color 0 0 0 0))
@@
     (stroke (width 0) (type default) (color 0 0 0 0))
   )
+  (wire (pts (xy 69.215 85.725) (xy 76.2 85.725))
+    (stroke (width 0) (type default) (color 0 0 0 0))
+  )
   (wire (pts (xy 91.44 46.99) (xy 89.535 46.99))
     (stroke (width 0) (type default) (color 0 0 0 0))
@@
     (stroke (width 0) (type default) (color 0 0 0 0))
   )
+  (wire (pts (xy 72.39 98.425) (xy 72.39 97.79))
+    (stroke (width 0) (type default) (color 0 0 0 0))
+  )
+  (wire (pts (xy 69.215 76.2) (xy 76.2 76.2))
+    (stroke (width 0) (type default) (color 0 0 0 0))
+  )
+  (wire (pts (xy 51.435 100.33) (xy 48.26 100.33))
+    (stroke (width 0) (type default) (color 0 0 0 0))
+  )
+  (wire (pts (xy 76.2 98.425) (xy 72.39 98.425))
+    (stroke (width 0) (type default) (color 0 0 0 0))
+  )
   (wire (pts (xy 103.505 61.595) (xy 103.505 40.005))
     (stroke (width 0) (type default) (color 0 0 0 0))
@@
     (stroke (width 0) (type default) (color 0 0 0 0))
   )
+  (wire (pts (xy 51.435 102.235) (xy 51.435 100.33))
+    (stroke (width 0) (type default) (color 0 0 0 0))
+  )
   (wire (pts (xy 114.3 46.99) (xy 114.3 48.26))
     (stroke (width 0) (type default) (color 0 0 0 0))
@@
     )
   )
+  (global_label "JTAG_TDO" (shape bidirectional) (at 69.215 76.2 180) (fields_autoplaced)
+    (effects (font (size 1.27 1.27)) (justify right))
+    (property "Intersheet References" "${INTERSHEET_REFS}" (id 0) (at 57.9724 76.1206 0)
+      (effects (font (size 1.27 1.27)) (justify right) hide)
+    )
+  )
   (global_label "3V3" (shape input) (at 126.365 47.625 90) (fields_autoplaced)
     (effects (font (size 1.27 1.27)) (justify left))
@@
     )
   )
+  (global_label "JTAG_TCK" (shape bidirectional) (at 69.215 73.025 180) (fields_autoplaced)
+    (effects (font (size 1.27 1.27)) (justify right))
+    (property "Intersheet References" "${INTERSHEET_REFS}" (id 0) (at 58.0329 72.9456 0)
+      (effects (font (size 1.27 1.27)) (justify right) hide)
+    )
+  )
   (global_label "3V3" (shape input) (at 76.835 47.625 90) (fields_autoplaced)
     (effects (font (size 1.27 1.27)) (justify left))
@@
     )
   )
+  (global_label "JTAG_TDI" (shape bidirectional) (at 69.215 69.85 180) (fields_autoplaced)
+    (effects (font (size 1.27 1.27)) (justify right))
+    (property "Intersheet References" "${INTERSHEET_REFS}" (id 0) (at 58.6981 69.7706 0)
+      (effects (font (size 1.27 1.27)) (justify right) hide)
+    )
+  )
+  (global_label "JTAG_TMS" (shape bidirectional) (at 69.215 66.675 180) (fields_autoplaced)
+    (effects (font (size 1.27 1.27)) (justify right))
+    (property "Intersheet References" "${INTERSHEET_REFS}" (id 0) (at 57.9119 66.5956 0)
+      (effects (font (size 1.27 1.27)) (justify right) hide)
+    )
+  )
+  (global_label "XTAL_N" (shape bidirectional) (at 69.215 82.55 180) (fields_autoplaced)
+    (effects (font (size 1.27 1.27)) (justify right))
+    (property "Intersheet References" "${INTERSHEET_REFS}" (id 0) (at 60.21 82.4706 0)
+      (effects (font (size 1.27 1.27)) (justify right) hide)
+    )
+  )
   (global_label "3V3" (shape input) (at 92.71 36.83 90) (fields_autoplaced)
     (effects (font (size 1.27 1.27)) (justify left))
@@
     )
   )
+  (global_label "XTAL_P" (shape bidirectional) (at 69.215 85.725 180) (fields_autoplaced)
+    (effects (font (size 1.27 1.27)) (justify right))
+    (property "Intersheet References" "${INTERSHEET_REFS}" (id 0) (at 60.2705 85.6456 0)
+      (effects (font (size 1.27 1.27)) (justify right) hide)
+    )
+  )
+  (global_label "3V3" (shape bidirectional) (at 46.99 67.945 90) (fields_autoplaced)
+    (effects (font (size 1.27 1.27)) (justify left))
+    (property "Intersheet References" "${INTERSHEET_REFS}" (id 0) (at 46.9106 62.0243 90)
+      (effects (font (size 1.27 1.27)) (justify left) hide)
+    )
+  )
   (symbol (lib_id "Device:C_Small") (at 111.76 43.815 0) (unit 1)
     (in_bom yes) (on_board yes)
@@
     (pin "2")
   )
+  (symbol (lib_id "Connector_Generic:Conn_01x03") (at 43.18 97.79 180) (unit 1)
+    (in_bom yes) (on_board yes) (fields_autoplaced)
+    (property "Reference" "J?" (id 0) (at 43.18 88.9 0))
+    (property "Value" "UART" (id 1) (at 43.18 91.44 0))
+    (property "Footprint" "Connector_PinSocket_2.54mm:PinSocket_1x03_P2.54mm_Vertical" (id 2) (at 43.18 97.79 0)
+      (effects (font (size 1.27 1.27)) hide)
+    )
+    (property "Datasheet" "~" (id 3) (at 43.18 97.79 0)
+      (effects (font (size 1.27 1.27)) hide)
+    )
+    (pin "1")
+    (pin "2")
+    (pin "3")
+  )
   (symbol (lib_id "power:GND") (at 95.25 114.3 0) (unit 1)
     (in_bom yes) (on_board yes) (fields_autoplaced)
@@
     (pin "2")
   )
+  (symbol (lib_id "Device:R_Small_US") (at 46.99 73.66 180) (unit 1)
+    (in_bom yes) (on_board yes) (fields_autoplaced)
+    (property "Reference" "R?" (id 0) (at 48.895 72.3899 0)
+      (effects (font (size 1.27 1.27)) (justify right))
+    )
+    (property "Value" "10k" (id 1) (at 48.895 74.9299 0)
+      (effects (font (size 1.27 1.27)) (justify right))
+    )
+    (property "Footprint" "Resistor_SMD:R_0805_2012Metric" (id 2) (at 46.99 73.66 0)
+      (effects (font (size 1.27 1.27)) hide)
+    )
+    (property "Datasheet" "~" (id 3) (at 46.99 73.66 0)
+      (effects (font (size 1.27 1.27)) hide)
+    )
+    (pin "1")
+    (pin "2")
+  )
   (symbol (lib_id "Device:C_Small") (at 91.44 43.815 0) (unit 1)
     (in_bom yes) (on_board yes) (fields_autoplaced)
@@
     (pin "9")
   )
+  (symbol (lib_id "power:GND") (at 51.435 102.235 0) (unit 1)
+    (in_bom yes) (on_board yes) (fields_autoplaced)
+    (property "Reference" "#PWR?" (id 0) (at 51.435 108.585 0)
+      (effects (font (size 1.27 1.27)) hide)
+    )
+    (property "Value" "GND" (id 1) (at 51.435 107.315 0)
+      (effects (font (size 1.27 1.27)) hide)
+    )
+    (property "Footprint" "" (id 2) (at 51.435 102.235 0)
+      (effects (font (size 1.27 1.27)) hide)
+    )
+    (property "Datasheet" "" (id 3) (at 51.435 102.235 0)
+      (effects (font (size 1.27 1.27)) hide)
+    )
+    (pin "1")
+  )
   (symbol (lib_id "Device:C_Small") (at 126.365 55.245 0) (unit 1)

Commit message: eod commit
Parts:
- removed C? (x3): 0.1uF, Capacitor_SMD:C_0603_1608Metric, symbol Device:C_Small
- removed C? (x3): 10uF, Capacitor_SMD:C_0603_1608Metric, symbol Device:C_Small
- added H1: MountingHole, MountingHole:MountingHole_2.5mm, symbol Mechanical:MountingHole
- added R2, R3, R4: 0, Resistor_SMD:R_0805_2012Metric, symbol Device:R_Small_US
- added R5, R6: 4.7k, Resistor_SMD:R_0805_2012Metric, symbol Device:R_Small_US
- added TP1, TP2: TestPoint, TestPoint:TestPoint_Pad_1.0x1.0mm, symbol Connector:TestPoint
- U1: renamed from U?; footprint Package_DFN_QFN:QFN-32-1EP_5x5mm_P0.5mm_EP3.7x3.7mm_ThermalVias -> Package_DFN_QFN:QFN-32-1EP_5x5mm_P0.5mm_EP3.3x3.3mm_ThermalVias
- gave numbers to parts that had none: 4
Connections:
- net 3V3: now also R5.2, R6.2
- net at J1.2 (Pin_2), U1.28 (U0TXD): now also R2.1, TP2.1
- net at J1.3 (Pin_3), U1.27 (U0RXD): now also R3.2, TP1.1
- net at U1.1 (LNA_IN): now also R4.2
- net I2C_SCL: now reaches U1.6 (GPIO2)
- net I2C_SCL: now also R5.1
- net I2C_SDA: now reaches U1.8 (GPIO3)
- net I2C_SDA: now also R6.1
- new net ANT: R4.1
- new net USB_DN: R3.1
- new net USB_DP: R2.2
- no-connect marks 16 -> 14
Other:
- moved on the sheet: C3, C4

Commit message: first layout rev
Parts:
- removed TP1, TP2: TestPoint, TestPoint:TestPoint_Pad_1.0x1.0mm, symbol Connector:TestPoint
Changed lines of the file:
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@@
   (junction (at 83.185 51.435) (diameter 0) (color 0 0 0 0)
   )
-  (junction (at 59.055 97.79) (diameter 0) (color 0 0 0 0)
-  )
   (junction (at 86.36 50.165) (diameter 0) (color 0 0 0 0)
   )
-  (junction (at 52.705 95.25) (diameter 0) (color 0 0 0 0)
-  )
   (junction (at 93.98 50.165) (diameter 0) (color 0 0 0 0)
   )
@@
     (stroke (width 0) (type default) (color 0 0 0 0))
   )
-  (wire (pts (xy 48.26 95.25) (xy 52.705 95.25))
+  (wire (pts (xy 48.26 95.25) (xy 66.04 95.25))
     (stroke (width 0) (type default) (color 0 0 0 0))
   )
@@
     (stroke (width 0) (type default) (color 0 0 0 0))
   )
-  (wire (pts (xy 59.055 92.71) (xy 59.055 97.79))
-    (stroke (width 0) (type default) (color 0 0 0 0))
-  )
   (wire (pts (xy 80.645 56.515) (xy 80.645 57.15))
     (stroke (width 0) (type default) (color 0 0 0 0))
@@
     (stroke (width 0) (type default) (color 0 0 0 0))
   )
-  (wire (pts (xy 59.055 97.79) (xy 48.26 97.79))
-    (stroke (width 0) (type default) (color 0 0 0 0))
-  )
   (wire (pts (xy 69.215 85.725) (xy 76.2 85.725))
     (stroke (width 0) (type default) (color 0 0 0 0))
@@
     (stroke (width 0) (type default) (color 0 0 0 0))
   )
-  (wire (pts (xy 52.705 95.25) (xy 66.04 95.25))
-    (stroke (width 0) (type default) (color 0 0 0 0))
-  )
   (wire (pts (xy 76.2 98.425) (xy 72.39 98.425))
     (stroke (width 0) (type default) (color 0 0 0 0))
@@
     (stroke (width 0) (type default) (color 0 0 0 0))
   )
-  (wire (pts (xy 52.705 92.71) (xy 52.705 95.25))
-    (stroke (width 0) (type default) (color 0 0 0 0))
-  )
   (wire (pts (xy 73.66 107.95) (xy 73.66 109.855))
     (stroke (width 0) (type default) (color 0 0 0 0))
@@
     (stroke (width 0) (type default) (color 0 0 0 0))
   )
-  (wire (pts (xy 62.865 97.79) (xy 59.055 97.79))
+  (wire (pts (xy 48.26 97.79) (xy 62.865 97.79))
     (stroke (width 0) (type default) (color 0 0 0 0))
   )
@@
     )
   )
-  (symbol (lib_id "Connector:TestPoint") (at 52.705 92.71 0) (unit 1)
-    (in_bom yes) (on_board yes)
-    (property "Reference" "TP1" (id 0) (at 53.975 89.535 0)
-      (effects (font (size 1.27 1.27)) (justify left))
-    )
-    (property "Value" "TestPoint" (id 1) (at 55.245 90.6779 0)
-      (effects (font (size 1.27 1.27)) (justify left) hide)
-    )
-    (property "Footprint" "TestPoint:TestPoint_Pad_1.0x1.0mm" (id 2) (at 57.785 92.71 0)
-      (effects (font (size 1.27 1.27)) hide)
-    )
-    (property "Datasheet" "~" (id 3) (at 57.785 92.71 0)
-      (effects (font (size 1.27 1.27)) hide)
-    )
-    (pin "1")
-  )
   (symbol (lib_id "Device:R_Small_US") (at 62.865 104.14 0) (unit 1)
     (in_bom yes) (on_board yes)
@@
     )
   )
-  (symbol (lib_id "Connector:TestPoint") (at 59.055 92.71 0) (unit 1)
-    (in_bom yes) (on_board yes)
-    (property "Reference" "TP2" (id 0) (at 60.325 89.535 0)
-      (effects (font (size 1.27 1.27)) (justify left))
-    )
-    (property "Value" "TestPoint" (id 1) (at 61.595 90.6779 0)
-      (effects (font (size 1.27 1.27)) (justify left) hide)
-    )
-    (property "Footprint" "TestPoint:TestPoint_Pad_1.0x1.0mm" (id 2) (at 64.135 92.71 0)
-      (effects (font (size 1.27 1.27)) hide)
-    )
-    (property "Datasheet" "~" (id 3) (at 64.135 92.71 0)
-      (effects (font (size 1.27 1.27)) hide)
-    )
-    (pin "1")
-  )
   (symbol (lib_id "Device:R_Small_US") (at 73.66 105.41 180) (unit 1)

Commit message: add bom
Other:
- company: (none) -> JCM
- title: (none) -> PortaNet
Changed lines of the file:
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@@
 (kicad_sch (version 20211123) (generator eeschema)
   (paper "A4")
+  (title_block
+    (title "PortaNet")
+    (date "2022-03-12")
+    (rev "1.0")
+    (company "JCM")
+  )
   (junction (at 139.7 66.675) (diameter 0) (color 0 0 0 0)
   )

Commit message: board v2 changes
Parts:
- removed R2, R3: 0, Resistor_SMD:R_0805_2012Metric, symbol Device:R_Small_US
- added C1: (no value), symbol Device:C_Small
- J1: value UART -> (none); footprint Connector_PinSocket_2.54mm:PinSocket_1x03_P2.54mm_Vertical -> (none); symbol Connector_Generic:Conn_01x03 -> Connector_Generic:Conn_01x04
Connections:
- net GND: now also C1.2
- net USB_DN: now also U1.25 (GPIO18)
- net USB_DP: now also U1.26 (GPIO19)
- net at R1.1, U1.7 (CHIP_EN): now also C1.1
- net JTAG_TCK: no longer names the net of U1.12 (MTCK)
- net JTAG_TDI: no longer names the net of U1.10 (MTDI)
- net JTAG_TDO: no longer names the net of U1.13 (MTDO)
- net JTAG_TMS: no longer names the net of U1.9 (MTMS)
- new net 5V: J1.4 (Pin_4)
- no-connect marks 14 -> 16
