File: hardware/kicad/PortaNet/esp32.kicad_sch (KiCad schematic)
At the start: 10 parts, among them U1 ESP32-C3

Commit message: updates
Parts:
- added C2: 0.1uF, Capacitor_SMD:C_0603_1608Metric, symbol Device:C_Small
- added J4: (no value), symbol Connector_Generic:Conn_01x02
- added R2, R3: (no value), symbol Device:R_Small_US
- C1: value (none) -> 1uF; footprint (none) -> Capacitor_SMD:C_0603_1608Metric
Connections:
- net 3V3: now also R2.2, R3.2
- net GND: now also C2.2, J4.2 (Pin_2)
- net I2C_SCL: now also U1.9 (MTMS); no longer U1.6 (GPIO2)
- net at U1.14 (GPIO8): now also R3.1
- net at U1.15 (GPIO9): now also C2.1, J4.1 (Pin_1)
- new net: R2.1, U1.6 (GPIO2)
- no-connect marks 16 -> 13
Other:
- moved on the sheet: R5

Commit message: add gerbers
Parts:
- added R11: (no value), symbol Device:R_Small_US
- J1: value (none) -> UART; footprint (none) -> Connector_PinSocket_2.54mm:PinSocket_1x04_P2.54mm_Vertical
- J4: value (none) -> RST; footprint (none) -> Connector_PinHeader_2.54mm:PinHeader_1x02_P2.54mm_Vertical
- R2, R3: value (none) -> 10k; footprint (none) -> Resistor_SMD:R_0805_2012Metric
Connections:
- net at U1.28 (U0TXD): now also R11.1; no longer J1.2 (Pin_2)
- new net: J1.2 (Pin_2), R11.2
Changed lines of the file:
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@@
     (stroke (width 0) (type default) (color 0 0 0 0))
   )
+  (wire (pts (xy 76.2 98.425) (xy 71.755 98.425))
+    (stroke (width 0) (type default) (color 0 0 0 0))
+  )
+  (wire (pts (xy 48.26 97.79) (xy 59.69 97.79))
+    (stroke (width 0) (type default) (color 0 0 0 0))
+  )
   (wire (pts (xy 106.68 50.165) (xy 109.855 50.165))
     (stroke (width 0) (type default) (color 0 0 0 0))
@@
     (stroke (width 0) (type default) (color 0 0 0 0))
   )
+  (wire (pts (xy 71.755 97.79) (xy 64.77 97.79))
+    (stroke (width 0) (type default) (color 0 0 0 0))
+  )
   (wire (pts (xy 69.215 85.725) (xy 76.2 85.725))
     (stroke (width 0) (type default) (color 0 0 0 0))
@@
     (stroke (width 0) (type default) (color 0 0 0 0))
   )
-  (wire (pts (xy 72.39 98.425) (xy 72.39 97.79))
-    (stroke (width 0) (type default) (color 0 0 0 0))
-  )
   (wire (pts (xy 103.505 50.165) (xy 103.505 61.595))
     (stroke (width 0) (type default) (color 0 0 0 0))
@@
     (stroke (width 0) (type default) (color 0 0 0 0))
   )
-  (wire (pts (xy 76.2 98.425) (xy 72.39 98.425))
-    (stroke (width 0) (type default) (color 0 0 0 0))
-  )
   (wire (pts (xy 138.43 73.025) (xy 138.43 64.77))
     (stroke (width 0) (type default) (color 0 0 0 0))
@@
     (stroke (width 0) (type default) (color 0 0 0 0))
   )
-  (wire (pts (xy 48.26 97.79) (xy 72.39 97.79))
-    (stroke (width 0) (type default) (color 0 0 0 0))
-  )
   (wire (pts (xy 80.645 57.15) (xy 83.185 57.15))
     (stroke (width 0) (type default) (color 0 0 0 0))
@@
     (stroke (width 0) (type default) (color 0 0 0 0))
   )
+  (wire (pts (xy 71.755 98.425) (xy 71.755 97.79))
+    (stroke (width 0) (type default) (color 0 0 0 0))
+  )
   (wire (pts (xy 150.495 76.2) (xy 167.005 76.2))
     (stroke (width 0) (type default) (color 0 0 0 0))
@@
     )
   )
+  (symbol (lib_id "Device:R_Small_US") (at 62.23 97.79 270) (unit 1)
+    (in_bom yes) (on_board yes)
+    (property "Reference" "R11" (id 0) (at 61.595 100.33 90))
+    (property "Value" "" (id 1) (at 62.23 102.235 90))
+    (property "Footprint" "" (id 2) (at 62.23 97.79 0)
+      (effects (font (size 1.27 1.27)) hide)
+    )
+    (property "Datasheet" "~" (id 3) (at 62.23 97.79 0)
+      (effects (font (size 1.27 1.27)) hide)
+    )
+    (pin "1")
+    (pin "2")
+  )
   (symbol (lib_id "Device:R_Small_US") (at 146.685 62.23 180) (unit 1)
     (in_bom yes) (on_board yes) (fields_autoplaced)
@@
     (in_bom yes) (on_board yes)
     (property "Reference" "J1" (id 0) (at 38.1 95.885 0))
-    (property "Value" "" (id 1) (at 38.1 97.79 0))
-    (property "Footprint" "" (id 2) (at 43.18 97.79 0)
+    (property "Value" "UART" (id 1) (at 38.1 97.79 0))
+    (property "Footprint" "Connector_PinSocket_2.54mm:PinSocket_1x04_P2.54mm_Vertical" (id 2) (at 43.18 97.79 0)
       (effects (font (size 1.27 1.27)) hide)
     )
@@
       (effects (font (size 1.27 1.27)) (justify right))
     )
-    (property "Value" "" (id 1) (at 140.335 63.4999 0)
+    (property "Value" "10k" (id 1) (at 140.335 63.4999 0)
       (effects (font (size 1.27 1.27)) (justify right))
     )
-    (property "Footprint" "" (id 2) (at 138.43 62.23 0)
+    (property "Footprint" "Resistor_SMD:R_0805_2012Metric" (id 2) (at 138.43 62.23 0)
       (effects (font (size 1.27 1.27)) hide)
     )
@@
       (effects (font (size 1.27 1.27)) (justify right))
     )
-    (property "Value" "" (id 1) (at 127 63.5 0)
+    (property "Value" "10k" (id 1) (at 127 63.5 0)
       (effects (font (size 1.27 1.27)) (justify right))
     )
-    (property "Footprint" "" (id 2) (at 132.08 62.23 0)
+    (property "Footprint" "Resistor_SMD:R_0805_2012Metric" (id 2) (at 132.08 62.23 0)
       (effects (font (size 1.27 1.27)) hide)
     )
@@
       (effects (font (size 1.27 1.27)) (justify right))
     )
-    (property "Value" "" (id 1) (at 172.72 72.3899 90)
+    (property "Value" "RST" (id 1) (at 172.72 72.3899 90)
       (effects (font (size 1.27 1.27)) (justify right))
     )
-    (property "Footprint" "" (id 2) (at 167.005 71.12 0)
+    (property "Footprint" "Connector_PinHeader_2.54mm:PinHeader_1x02_P2.54mm_Vertical" (id 2) (at 167.005 71.12 0)
       (effects (font (size 1.27 1.27)) hide)
     )

Commit message: simplify
Parts:
- removed J1: UART, Connector_PinSocket_2.54mm:PinSocket_1x04_P2.54mm_Vertical, symbol Connector_Generic:Conn_01x04
- removed R11: (no value), symbol Device:R_Small_US
- removed R4: 0, Resistor_SMD:R_0805_2012Metric, symbol Device:R_Small_US
- removed R5, R6: 4.7k, Resistor_SMD:R_0805_2012Metric, symbol Device:R_Small_US
Connections:
- net ANT: now also U1.1 (LNA_IN)
- net I2C_SCL: no longer names the net of U1.9 (MTMS)
- net I2C_SDA: no longer names the net of U1.8 (GPIO3)
- no-connect marks 13 -> 17

Commit message: v4
Parts:
- removed H1: MountingHole, MountingHole:MountingHole_2.5mm, symbol Mechanical:MountingHole
- removed J4: RST, Connector_PinHeader_2.54mm:PinHeader_1x02_P2.54mm_Vertical, symbol Connector_Generic:Conn_01x02
- added C13, C7: 0.1uF, Capacitor_SMD:C_0603_1608Metric, symbol Device:C_Small
- added C14, C8: 10uF, Capacitor_SMD:C_0603_1608Metric, symbol Device:C_Small
- added SW1: (no value), symbol Switch:SW_SPST
Connections:
- net 3V3: now also C13.1, C14.1, C7.1, C8.1
- net GND: now also C13.2, C14.2, C7.2, C8.2, SW1.2 (B)
- net at C2.1, U1.15 (GPIO9): now also SW1.1 (A)
Other:
- company: JCM -> (none)
- moved on the sheet: R2

Commit message: init commit
Parts:
- C2: value 0.1uF -> NC
- SW1: value (none) -> 434133025816; footprint (none) -> Button_Switch_SMD:SW_Push_1P1T_NO_Vertical_Wuerth_434133025816
- U1: value ESP32-C3 -> ESP32-C3FH4
Changed lines of the file:
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@@
     (title "PortaNet")
     (date "2022-05-01")
-    (rev "4.0")
+    (rev "4.1")
   )
   (junction (at 100.33 50.165) (diameter 0) (color 0 0 0 0)
@@
       (effects (font (size 1.27 1.27)) (justify left))
     )
-    (property "Value" "0.1uF" (id 1) (at 152.4 81.915 0)
+    (property "Value" "NC" (id 1) (at 152.4 81.915 0)
       (effects (font (size 1.27 1.27)) (justify left))
     )
@@
       (effects (font (size 1.27 1.27)) (justify left))
     )
-    (property "Value" "ESP32-C3" (id 1) (at 92.075 102.235 0)
+    (property "Value" "ESP32-C3FH4" (id 1) (at 92.71 102.235 0)
       (effects (font (size 1.27 1.27)) (justify left))
     )
@@
     (in_bom yes) (on_board yes)
     (property "Reference" "SW1" (id 0) (at 160.655 73.025 0))
-    (property "Value" "" (id 1) (at 160.655 72.39 0)
+    (property "Value" "434133025816" (id 1) (at 160.655 72.39 0)
       (effects (font (size 1.27 1.27)) hide)
     )
-    (property "Footprint" "" (id 2) (at 160.655 76.2 0)
+    (property "Footprint" "Button_Switch_SMD:SW_Push_1P1T_NO_Vertical_Wuerth_434133025816" (id 2) (at 160.655 76.2 0)
       (effects (font (size 1.27 1.27)) hide)
     )
