File: hardware/kicad/PortaNet/misc1.kicad_sch (KiCad schematic)
At the start: 3 parts

Commit message: eod commit
Parts:
- added C? (x2): 7pF, Capacitor_SMD:C_0603_1608Metric, symbol Device:C_Small
- added D?: L196L-UEC-TR, LED_SMD:LED_0603_1608Metric, symbol Device:LED
- added D?: L196L-QYC-TR, LED_SMD:LED_0603_1608Metric, symbol Device:LED
- added D? (x2): DSS13UTR, Diode_SMD:D_SOD-123F, symbol Device:D_Schottky
- added J?: Molex 0480370001, JoesFootprints:Molex_0480370001, symbol Connector:USB_A
- added J?: GRPB052VWVN-RC, Connector_PinHeader_1.27mm:PinHeader_2x05_P1.27mm_Vertical, symbol Connector:Conn_ARM_JTAG_SWD_10
- added R? (x2): 1k, Resistor_SMD:R_0805_2012Metric, symbol Device:R_Small_US
- added R? (x2): 22, Resistor_SMD:R_0805_2012Metric, symbol Device:R_Small_US
- added Y?: FL400WFQA1, Crystal:Crystal_SMD_3225-4Pin_3.2x2.5mm, symbol Device:Crystal_GND24
Connections:
- net 3V3: now also R?.2
- net 5V: now also D?.1 (K), D?.1 (K), R?.2
- net GND: now also C?.2, C?.2, D?.1 (K), D?.1 (K), J?.3 (GND), J?.4 (GND), J?.5 (GND), J?.5 (Shield), J?.9 (GNDDetect), Y?.2, Y?.4
- new net: D?.2 (A), R?.1 (x2)
- new net: D?.2 (A), J?.1 (VBUS)
- new net: J?.2 (D-), R?.1
- new net: J?.3 (D+), R?.1
- new net: D?.2 (A), J?.1 (VTref)
- new net JTAG_TCK: J?.4 (SWDCLK/TCK)
- new net JTAG_TDI: J?.8 (NC/TDI)
- new net JTAG_TDO: J?.6 (SWO/TDO)
- new net JTAG_TMS: J?.2 (SWDIO/TMS)
- new net USB_DN: R?.2
- new net USB_DP: R?.2
- new net XTAL_N: C?.1, Y?.1
- new net XTAL_P: C?.1, Y?.3
- no-connect marks 0 -> 1
Other:
- note added: "3.3V Regulator"
- note added: "Crystal"
- note added: "JTAG"
- note added: "LED Indicators"
- note added: "Male USB A Connector"

Commit message: eod commit
Parts:
- added AE1: ANT3216LL00R2400A, JoesFootprints:ANT3216LL00R2400A, symbol Device:Antenna_Shield
- added J3: OLED_PINS, JoesFootprints:OLED_0.91in_i2c, symbol Connector_Generic:Conn_01x04
- added TP3, TP4, TP5: TestPoint, TestPoint:TestPoint_Pad_1.0x1.0mm, symbol Connector:TestPoint
- gave numbers to parts that had none: 16
Connections:
- net 3V3: now also D4.1 (K), J3.2 (Pin_2), TP4.1
- net 5V: now also TP3.1; no longer D4.1 (K)
- net GND: now also J3.1 (Pin_1), TP5.1
- new net ANT: AE1.1 (A)
- new net I2C_SCL: J3.3 (Pin_3)
- new net I2C_SDA: J3.4 (Pin_4)
- no-connect marks 1 -> 2
Other:
- note added: "Antenna"
- note added: "I2C OLED"

Commit message: add bom
Other:
- company: (none) -> JCM
- title: (none) -> PortaNet
Changed lines of the file:
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@@
 (kicad_sch (version 20211123) (generator eeschema)
   (paper "A4")
+  (title_block
+    (title "PortaNet")
+    (date "2022-03-12")
+    (rev "1.0")
+    (company "JCM")
+  )
   (junction (at 62.865 29.21) (diameter 0) (color 0 0 0 0)
   )

Commit message: board v2 changes
Parts:
- removed D4: DSS13UTR, Diode_SMD:D_SOD-123F, symbol Device:D_Schottky
- removed J4: GRPB052VWVN-RC, Connector_PinHeader_1.27mm:PinHeader_2x05_P1.27mm_Vertical, symbol Connector:Conn_ARM_JTAG_SWD_10
Connections:
- no-connect marks 2 -> 1
Other:
- note removed: "JTAG"
Changed lines of the file:
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@@
   (junction (at 36.195 63.5) (diameter 0) (color 0 0 0 0)
   )
-  (junction (at 220.345 32.385) (diameter 0) (color 0 0 0 0)
-  )
   (junction (at 31.75 29.21) (diameter 0) (color 0 0 0 0)
   )
@@
   )
   (no_connect (at 166.37 73.025))
-  (no_connect (at 247.015 45.085))
   (wire (pts (xy 46.355 68.58) (xy 46.355 71.12))
     (stroke (width 0) (type default) (color 0 0 0 0))
@@
     (stroke (width 0) (type default) (color 0 0 0 0))
   )
-  (wire (pts (xy 254.635 32.385) (xy 259.08 32.385))
-    (stroke (width 0) (type default) (color 0 0 0 0))
-  )
   (wire (pts (xy 29.21 36.195) (xy 29.21 36.83))
     (stroke (width 0) (type default) (color 0 0 0 0))
@@
     (stroke (width 0) (type default) (color 0 0 0 0))
   )
-  (wire (pts (xy 266.7 32.385) (xy 269.875 32.385))
-    (stroke (width 0) (type default) (color 0 0 0 0))
-  )
   (wire (pts (xy 29.21 29.21) (xy 31.75 29.21))
     (stroke (width 0) (type default) (color 0 0 0 0))
@@
     (stroke (width 0) (type default) (color 0 0 0 0))
   )
-  (wire (pts (xy 220.345 29.845) (xy 220.345 32.385))
-    (stroke (width 0) (type default) (color 0 0 0 0))
-  )
   (wire (pts (xy 31.75 27.305) (xy 31.75 29.21))
     (stroke (width 0) (type default) (color 0 0 0 0))
@@
     (stroke (width 0) (type default) (color 0 0 0 0))
   )
-  (wire (pts (xy 239.395 45.085) (xy 239.395 48.895))
-    (stroke (width 0) (type default) (color 0 0 0 0))
-  )
-  (wire (pts (xy 234.315 45.085) (xy 234.315 48.895))
-    (stroke (width 0) (type default) (color 0 0 0 0))
-  )
   (wire (pts (xy 103.505 71.755) (xy 108.585 71.755))
     (stroke (width 0) (type default) (color 0 0 0 0))
@@
     (stroke (width 0) (type default) (color 0 0 0 0))
   )
-  (polyline (pts (xy 194.945 63.5) (xy 285.115 63.5))
-    (stroke (width 0) (type default) (color 0 0 0 0))
-  )
-  (wire (pts (xy 224.155 29.845) (xy 220.345 29.845))
-    (stroke (width 0) (type default) (color 0 0 0 0))
-  )
-  (wire (pts (xy 241.935 45.085) (xy 241.935 48.895))
-    (stroke (width 0) (type default) (color 0 0 0 0))
-  )
   (wire (pts (xy 113.665 28.575) (xy 120.65 28.575))
     (stroke (width 0) (type default) (color 0 0 0 0))
@@
     (stroke (width 0) (type default) (color 0 0 0 0))
   )
-  (wire (pts (xy 220.345 32.385) (xy 224.155 32.385))
-    (stroke (width 0) (type default) (color 0 0 0 0))
-  )
   (polyline (pts (xy 76.2 12.065) (xy 76.2 48.895))
     (stroke (width 0) (type default) (color 0 0 0 0))
@@
     (stroke (width 0) (type default) (color 0 0 0 0))
   )
-  (wire (pts (xy 220.345 32.385) (xy 220.345 33.655))
-    (stroke (width 0) (type default) (color 0 0 0 0))
-  )
   (polyline (pts (xy 76.2 80.645) (xy 138.43 80.645))
     (stroke (width 0) (type default) (color 0 0 0 0))
@@
   )
   (polyline (pts (xy 76.2 55.88) (xy 76.2 80.645))
-    (stroke (width 0) (type default) (color 0 0 0 0))
-  )
-  (wire (pts (xy 236.855 45.085) (xy 236.855 48.895))
     (stroke (width 0) (type default) (color 0 0 0 0))
   )
@@
     (effects (font (size 1.27 1.27)) (justify left bottom))
   )
-  (text "JTAG" (at 196.85 15.24 0)
-    (effects (font (size 1.27 1.27)) (justify left bottom))
-  )
   (text "I2C OLED" (at 127.635 79.375 0)
     (effects (font (size 1.27 1.27)) (justify left bottom))
   )
-  (global_label "JTAG_TMS" (shape bidirectional) (at 239.395 48.895 270) (fields_autoplaced)
-    (effects (font (size 1.27 1.27)) (justify right))
-    (property "Intersheet References" "${INTERSHEET_REFS}" (id 0) (at 239.3156 60.1981 90)
-      (effects (font (size 1.27 1.27)) (justify right) hide)
-    )
-  )
   (global_label "USB_DN" (shape bidirectional) (at 120.65 31.115 0) (fields_autoplaced)
     (effects (font (size 1.27 1.27)) (justify left))
     (property "Intersheet References" "${INTERSHEET_REFS}" (id 0) (at 130.4412 31.0356 0)
-      (effects (font (size 1.27 1.27)) (justify left) hide)
-    )
-  )
-  (global_label "3V3" (shape bidirectional) (at 269.875 32.385 0) (fields_autoplaced)
-    (effects (font (size 1.27 1.27)) (justify left))
-    (property "Intersheet References" "${INTERSHEET_REFS}" (id 0) (at 275.7957 32.3056 0)
       (effects (font (size 1.27 1.27)) (justify left) hide)
     )
@@
     )
   )
-  (global_label "JTAG_TCK" (shape bidirectional) (at 241.935 48.895 270) (fields_autoplaced)
-    (effects (font (size 1.27 1.27)) (justify right))
-    (property "Intersheet References" "${INTERSHEET_REFS}" (id 0) (at 241.8556 60.0771 90)
-      (effects (font (size 1.27 1.27)) (justify right) hide)
-    )
-  )
   (global_label "I2C_SCL" (shape input) (at 109.855 66.675 0) (fields_autoplaced)
     (effects (font (size 1.27 1.27)) (justify left))
@@
     )
   )
-  (global_label "JTAG_TDI" (shape bidirectional) (at 234.315 48.895 270) (fields_autoplaced)
-    (effects (font (size 1.27 1.27)) (justify right))
-    (property "Intersheet References" "${INTERSHEET_REFS}" (id 0) (at 234.2356 59.4119 90)
-      (effects (font (size 1.27 1.27)) (justify right) hide)
-    )
-  )
   (global_label "ANT" (shape bidirectional) (at 155.575 73.025 180) (fields_autoplaced)
     (effects (font (size 1.27 1.27)) (justify right))
@@
     )
   )
-  (global_label "JTAG_TDO" (shape bidirectional) (at 236.855 48.895 270) (fields_autoplaced)
-    (effects (font (size 1.27 1.27)) (justify right))
-    (property "Intersheet References" "${INTERSHEET_REFS}" (id 0) (at 236.7756 60.1376 90)
-      (effects (font (size 1.27 1.27)) (justify right) hide)
-    )
-  )
   (global_label "5V" (shape input) (at 152.4 19.05 180) (fields_autoplaced)
     (effects (font (size 1.27 1.27)) (justify right))
@@
     (pin "2")
   )
-  (symbol (lib_id "power:GND") (at 220.345 33.655 0) (mirror y) (unit 1)
-    (in_bom yes) (on_board yes) (fields_autoplaced)
-    (property "Reference" "#PWR0116" (id 0) (at 220.345 40.005 0)
-      (effects (font (size 1.27 1.27)) hide)
-    )
-    (property "Value" "GND" (id 1) (at 220.345 38.1 0)
-      (effects (font (size 1.27 1.27)) hide)
-    )
-    (property "Footprint" "" (id 2) (at 220.345 33.655 0)
-      (effects (font (size 1.27 1.27)) hide)
-    )
-    (property "Datasheet" "" (id 3) (at 220.345 33.655 0)
-      (effects (font (size 1.27 1.27)) hide)
-    )
-    (pin "1")
-  )
   (symbol (lib_id "Device:D_Schottky") (at 111.76 23.495 180) (unit 1)
     (in_bom yes) (on_board yes)
@@
     (pin "2")
   )
-  (symbol (lib_id "Connector:Conn_ARM_JTAG_SWD_10") (at 239.395 32.385 270) (unit 1)
-    (in_bom yes) (on_board yes) (fields_autoplaced)
-    (property "Reference" "J4" (id 0) (at 239.395 17.145 90))
-    (property "Value" "GRPB052VWVN-RC" (id 1) (at 239.395 19.685 90))
-    (property "Footprint" "Connector_PinHeader_1.27mm:PinHeader_2x05_P1.27mm_Vertical" (id 2) (at 239.395 32.385 0)
-      (effects (font (size 1.27 1.27)) hide)
-    )
-    (property "Datasheet" "https://www.digikey.com/en/products/detail/sullins-connector-solutions/GRPB052VWVN-RC/1786455" (id 3) (at 207.645 23.495 90)
-      (effects (font (size 1.27 1.27)) hide)
-    )
-    (pin "1")
-    (pin "10")
-    (pin "2")
-    (pin "3")
-    (pin "4")
-    (pin "5")
-    (pin "6")
-    (pin "7")
-    (pin "8")
-    (pin "9")
-  )
   (symbol (lib_id "power:GND") (at 108.585 74.295 0) (unit 1)
     (in_bom yes) (on_board yes) (fields_autoplaced)
@@
       (effects (font (size 1.27 1.27)) hide)
     )
-    (pin "1")
-    (pin "2")
-  )
-  (symbol (lib_id "Device:D_Schottky") (at 262.89 32.385 180) (unit 1)
-    (in_bom yes) (on_board yes)
-    (property "Reference" "D4" (id 0) (at 262.89 27.94 0))
-    (property "Value" "DSS13UTR" (id 1) (at 263.525 29.845 0))
-    (property "Footprint" "Diode_SMD:D_SOD-123F" (id 2) (at 262.89 32.385 0)
-      (effects (font (size 1.27 1.27)) hide)
-    )
-    (property "Datasheet" "https://www.digikey.com/en/products/detail/smc-diode-solutions/DSS13UTR/8341858" (id 3) (at 262.89 32.385 0)
-      (effects (font (size 1.27 1.27)) hide)
-    )

Commit message: simplify
Parts:
- removed AE1: ANT3216LL00R2400A, JoesFootprints:ANT3216LL00R2400A, symbol Device:Antenna_Shield
- removed D2: L196L-UEC-TR, LED_SMD:LED_0603_1608Metric, symbol Device:LED
- removed D3: L196L-QYC-TR, LED_SMD:LED_0603_1608Metric, symbol Device:LED
- removed J3: OLED_PINS, JoesFootprints:OLED_0.91in_i2c, symbol Connector_Generic:Conn_01x04
- removed R10, R9: 1k, Resistor_SMD:R_0805_2012Metric, symbol Device:R_Small_US
- removed TP3, TP4, TP5: TestPoint, TestPoint:TestPoint_Pad_1.0x1.0mm, symbol Connector:TestPoint
- added C5, C6: (no value), symbol Device:C_Small
- added J1: (no value), symbol Connector:Conn_Coaxial
- added L1: (no value), symbol Device:L
Connections:
- net ANT: now also C5.1, L1.1
- net GND: now also C5.2, C6.2, J1.2 (Ext)
- new net: C6.1, J1.1 (In), L1.2
- no-connect marks 1 -> 0
Other:
- note removed: "I2C OLED"
- note removed: "LED Indicators"
