File: hardware/kicad/PortaNet/misc1.kicad_sch (KiCad schematic)
At the start: 14 parts, among them J2 Molex 0480370001, U2 AP2114HA-3.3TRG1, Y1 FL400WFQA1

Commit message: v4
Parts:
- removed R7, R8: 22, Resistor_SMD:R_0805_2012Metric, symbol Device:R_Small_US
- added R4, R5: (no value), symbol Device:R_Small_US
- C5, C6: value (none) -> TBD; footprint (none) -> Capacitor_SMD:C_0603_1608Metric
- J1: value (none) -> SMA
Connections:
- net GND: no longer J2.5 (Shield)
- net USB_DN: now also R5.1
- net USB_DP: now also R4.1
- net D-: now reaches J2.2 (D-)
- net D-: now also R5.2
- net D+: now reaches J2.3 (D+)
- net D+: now also R4.2
- no-connect marks 0 -> 1
Other:
- company: JCM -> (none)
Changed lines of the file:
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@@
   (title_block
     (title "PortaNet")
-    (date "2022-03-12")
-    (rev "1.0")
-    (company "JCM")
+    (date "2022-05-01")
+    (rev "4.0")
   )
   (junction (at 56.515 63.5) (diameter 0) (color 0 0 0 0)
@@
   (junction (at 34.29 29.21) (diameter 0) (color 0 0 0 0)
   )
+  (no_connect (at 92.71 38.735))
+  (wire (pts (xy 102.87 31.115) (xy 109.855 31.115))
+    (stroke (width 0) (type default) (color 0 0 0 0))
+  )
   (wire (pts (xy 46.355 68.58) (xy 46.355 71.12))
     (stroke (width 0) (type default) (color 0 0 0 0))
@@
     (stroke (width 0) (type default) (color 0 0 0 0))
   )
-  (wire (pts (xy 92.71 40.005) (xy 92.71 38.735))
-    (stroke (width 0) (type default) (color 0 0 0 0))
-  )
   (wire (pts (xy 31.75 36.83) (xy 31.75 37.465))
     (stroke (width 0) (type default) (color 0 0 0 0))
@@
     (stroke (width 0) (type default) (color 0 0 0 0))
   )
-  (wire (pts (xy 90.17 40.64) (xy 90.17 40.005))
+  (wire (pts (xy 114.935 31.115) (xy 120.65 31.115))
     (stroke (width 0) (type default) (color 0 0 0 0))
   )
@@
     (stroke (width 0) (type default) (color 0 0 0 0))
   )
-  (wire (pts (xy 90.17 40.005) (xy 92.71 40.005))
-    (stroke (width 0) (type default) (color 0 0 0 0))
-  )
-  (wire (pts (xy 102.87 31.115) (xy 108.585 31.115))
-    (stroke (width 0) (type default) (color 0 0 0 0))
-  )
   (wire (pts (xy 147.32 43.18) (xy 157.48 43.18))
     (stroke (width 0) (type default) (color 0 0 0 0))
@@
     (stroke (width 0) (type default) (color 0 0 0 0))
   )
-  (wire (pts (xy 113.665 31.115) (xy 120.65 31.115))
-    (stroke (width 0) (type default) (color 0 0 0 0))
-  )
   (wire (pts (xy 56.515 70.485) (xy 56.515 72.39))
     (stroke (width 0) (type default) (color 0 0 0 0))
@@
     (stroke (width 0) (type default) (color 0 0 0 0))
   )
-  (wire (pts (xy 113.665 28.575) (xy 120.65 28.575))
+  (wire (pts (xy 102.87 28.575) (xy 109.855 28.575))
     (stroke (width 0) (type default) (color 0 0 0 0))
   )
@@
     (stroke (width 0) (type default) (color 0 0 0 0))
   )
+  (wire (pts (xy 114.935 28.575) (xy 120.65 28.575))
+    (stroke (width 0) (type default) (color 0 0 0 0))
+  )
   (wire (pts (xy 56.515 63.5) (xy 56.515 65.405))
     (stroke (width 0) (type default) (color 0 0 0 0))
@@
   )
   (wire (pts (xy 34.29 29.21) (xy 34.29 31.115))
-    (stroke (width 0) (type default) (color 0 0 0 0))
-  )
-  (wire (pts (xy 102.87 28.575) (xy 108.585 28.575))
     (stroke (width 0) (type default) (color 0 0 0 0))
   )
@@
   )
   (text "Crystal" (at 13.335 52.705 0)
+    (effects (font (size 1.27 1.27)) (justify left bottom))
+  )
+  (label "D-" (at 104.775 31.115 0)
+    (effects (font (size 1.27 1.27)) (justify left bottom))
+  )
+  (label "D+" (at 104.775 28.575 0)
     (effects (font (size 1.27 1.27)) (justify left bottom))
   )
@@
     (pin "2")
   )
-  (symbol (lib_id "power:GND") (at 90.17 40.64 0) (mirror y) (unit 1)
-    (in_bom yes) (on_board yes) (fields_autoplaced)
-    (property "Reference" "#PWR0109" (id 0) (at 90.17 46.99 0)
-      (effects (font (size 1.27 1.27)) hide)
-    )
-    (property "Value" "GND" (id 1) (at 90.17 45.085 0)
-      (effects (font (size 1.27 1.27)) hide)
-    )
-    (property "Footprint" "" (id 2) (at 90.17 40.64 0)
-      (effects (font (size 1.27 1.27)) hide)
-    )
-    (property "Datasheet" "" (id 3) (at 90.17 40.64 0)
-      (effects (font (size 1.27 1.27)) hide)
-    )
-    (pin "1")
-  )
   (symbol (lib_id "Connector:Conn_Coaxial") (at 189.23 43.18 0) (unit 1)
     (in_bom yes) (on_board yes)
@@
       (effects (font (size 1.27 1.27)) (justify left))
     )
-    (property "Value" "" (id 1) (at 186.055 40.005 0)
+    (property "Value" "SMA" (id 1) (at 186.055 40.005 0)
       (effects (font (size 1.27 1.27)) (justify left))
     )
@@
     (pin "2")
   )
-  (symbol (lib_id "Device:R_Small_US") (at 111.125 28.575 90) (unit 1)
-    (in_bom yes) (on_board yes)
-    (property "Reference" "R7" (id 0) (at 113.665 27.305 90))
-    (property "Value" "22" (id 1) (at 107.95 27.305 90))
-    (property "Footprint" "Resistor_SMD:R_0805_2012Metric" (id 2) (at 111.125 28.575 0)
-      (effects (font (size 1.27 1.27)) hide)
-    )
-    (property "Datasheet" "~" (id 3) (at 111.125 28.575 0)
-      (effects (font (size 1.27 1.27)) hide)
-    )
-    (pin "1")
-    (pin "2")
-  )
-  (symbol (lib_id "Device:R_Small_US") (at 111.125 31.115 90) (unit 1)
-    (in_bom yes) (on_board yes)
-    (property "Reference" "R8" (id 0) (at 113.665 32.385 90))
-    (property "Value" "22" (id 1) (at 108.585 32.385 90))
-    (property "Footprint" "Resistor_SMD:R_0805_2012Metric" (id 2) (at 111.125 31.115 0)
-      (effects (font (size 1.27 1.27)) hide)
-    )
-    (property "Datasheet" "~" (id 3) (at 111.125 31.115 0)
+  (symbol (lib_id "Device:R_Small_US") (at 112.395 31.115 270) (unit 1)
+    (in_bom yes) (on_board yes)
+    (property "Reference" "R5" (id 0) (at 115.57 33.655 90)
+      (effects (font (size 1.27 1.27)) (justify right))
+    )
+    (property "Value" "" (id 1) (at 110.49 33.02 90)
+      (effects (font (size 1.27 1.27)) (justify right))
+    )
+    (property "Footprint" "" (id 2) (at 112.395 31.115 0)
+      (effects (font (size 1.27 1.27)) hide)
+    )
+    (property "Datasheet" "~" (id 3) (at 112.395 31.115 0)
+      (effects (font (size 1.27 1.27)) hide)
+    )
+    (pin "1")
+    (pin "2")
+  )
+  (symbol (lib_id "Device:R_Small_US") (at 112.395 28.575 270) (unit 1)
+    (in_bom yes) (on_board yes)
+    (property "Reference" "R4" (id 0) (at 115.57 26.67 90)
+      (effects (font (size 1.27 1.27)) (justify right))
+    )
+    (property "Value" "" (id 1) (at 110.49 26.67 90)
+      (effects (font (size 1.27 1.27)) (justify right))
+    )
+    (property "Footprint" "" (id 2) (at 112.395 28.575 0)
+      (effects (font (size 1.27 1.27)) hide)
+    )
+    (property "Datasheet" "~" (id 3) (at 112.395 28.575 0)
       (effects (font (size 1.27 1.27)) hide)
     )
@@
       (effects (font (size 1.27 1.27)) (justify left))
     )
-    (property "Value" "" (id 1) (at 152.4 50.165 0)
-      (effects (font (size 1.27 1.27)) (justify left))
-    )
-    (property "Footprint" "" (id 2) (at 157.48 48.26 0)
+    (property "Value" "TBD" (id 1) (at 152.4 50.165 0)
+      (effects (font (size 1.27 1.27)) (justify left))
+    )
+    (property "Footprint" "Capacitor_SMD:C_0603_1608Metric" (id 2) (at 157.48 48.26 0)
       (effects (font (size 1.27 1.27)) hide)
     )
@@
       (effects (font (size 1.27 1.27)) (justify left))
     )
-    (property "Value" "" (id 1) (at 174.625 50.165 0)
-      (effects (font (size 1.27 1.27)) (justify left))
-    )
-    (property "Footprint" "" (id 2) (at 179.705 48.26 0)
-      (effects (font (size 1.27 1.27)) hide)
-    )
+    (property "Value" "TBD" (id 1) (at 174.625 50.165 0)
+      (effects (font (size 1.27 1.27)) (justify left))
+    )
+    (property "Footprint" "Capacitor_SMD:C_0603_1608Metric" (id 2) (at 179.705 48.26 0)
+      (effects (font (size 1.27 1.27)) hide)
+    )

Commit message: init commit
Parts:
- J1: footprint (none) -> Connector_Coaxial:SMA_Amphenol_132134_Vertical
- L1: value (none) -> TBD; footprint (none) -> Inductor_SMD:L_0805_2012Metric_Pad1.15x1.40mm_HandSolder
- R4, R5: value (none) -> 22; footprint (none) -> Resistor_SMD:R_0805_2012Metric
Other:
- note added: "DEFAULT: NC"
- note added: "DEFAULT: SHORT"
Changed lines of the file:
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@@
     (title "PortaNet")
     (date "2022-05-01")
-    (rev "4.0")
+    (rev "4.1")
   )
   (junction (at 56.515 63.5) (diameter 0) (color 0 0 0 0)
@@
     (effects (font (size 1.27 1.27)) (justify left bottom))
   )
+  (text "DEFAULT: SHORT" (at 161.925 35.56 0)
+    (effects (font (size 1 1)) (justify left bottom))
+  )
   (text "3.3V Regulator" (at 12.7 14.605 0)
     (effects (font (size 1.27 1.27)) (justify left bottom))
@@
     (effects (font (size 1.27 1.27)) (justify left bottom))
   )
+  (text "DEFAULT: NC" (at 169.545 53.34 0)
+    (effects (font (size 1 1)) (justify left bottom))
+  )
   (text "Crystal" (at 13.335 52.705 0)
     (effects (font (size 1.27 1.27)) (justify left bottom))
+  )
+  (text "DEFAULT: NC" (at 143.51 53.975 0)
+    (effects (font (size 1 1)) (justify left bottom))
   )
   (label "D-" (at 104.775 31.115 0)
@@
     (in_bom yes) (on_board yes) (fields_autoplaced)
     (property "Reference" "L1" (id 0) (at 168.275 36.83 90))
-    (property "Value" "" (id 1) (at 168.275 39.37 90))
-    (property "Footprint" "" (id 2) (at 168.275 43.18 0)
+    (property "Value" "TBD" (id 1) (at 168.275 39.37 90))
+    (property "Footprint" "Inductor_SMD:L_0805_2012Metric_Pad1.15x1.40mm_HandSolder" (id 2) (at 168.275 43.18 0)
       (effects (font (size 1.27 1.27)) hide)
     )
@@
       (effects (font (size 1.27 1.27)) (justify left))
     )
-    (property "Footprint" "" (id 2) (at 189.23 43.18 0)
+    (property "Footprint" "Connector_Coaxial:SMA_Amphenol_132134_Vertical" (id 2) (at 189.23 43.18 0)
       (effects (font (size 1.27 1.27)) hide)
     )
@@
       (effects (font (size 1.27 1.27)) (justify right))
     )
-    (property "Value" "" (id 1) (at 110.49 33.02 90)
+    (property "Value" "22" (id 1) (at 110.49 33.02 90)
       (effects (font (size 1.27 1.27)) (justify right))
     )
-    (property "Footprint" "" (id 2) (at 112.395 31.115 0)
+    (property "Footprint" "Resistor_SMD:R_0805_2012Metric" (id 2) (at 112.395 31.115 0)
       (effects (font (size 1.27 1.27)) hide)
     )
@@
       (effects (font (size 1.27 1.27)) (justify right))
     )
-    (property "Value" "" (id 1) (at 110.49 26.67 90)
+    (property "Value" "22" (id 1) (at 110.49 26.67 90)
       (effects (font (size 1.27 1.27)) (justify right))
     )
-    (property "Footprint" "" (id 2) (at 112.395 28.575 0)
-      (effects (font (size 1.27 1.27)) hide)
-    )
+    (property "Footprint" "Resistor_SMD:R_0805_2012Metric" (id 2) (at 112.395 28.575 0)
+      (effects (font (size 1.27 1.27)) hide)
+    )
