File: hardware/kicad/PortaNet/PortaNet.kicad_sch (KiCad schematic)
At the start: 0 parts

Commit message: v4
Other:
- company: JCM -> (none)
Changed lines of the file:
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@@
   (title_block
     (title "PortaNet")
-    (date "2022-03-12")
-    (rev "1.0")
-    (company "JCM")
+    (date "2022-05-01")
+    (rev "4.0")
   )
   (text "Miscellaneous Hardware" (at 36.195 53.34 0)
@@
       (reference "#PWR02") (unit 1) (value "GND") (footprint "")
     )
+    (path "/1e5d0253-acc2-4f0d-86a2-9343225c71a7/f83f6daf-16e2-4342-8acf-e431395a8020"
+      (reference "#PWR03") (unit 1) (value "GND") (footprint "")
+    )
     (path "/1e5d0253-acc2-4f0d-86a2-9343225c71a7/845b399e-676e-463f-8468-615daa2923c9"
       (reference "#PWR0101") (unit 1) (value "GND") (footprint "")
@@
       (reference "#PWR0108") (unit 1) (value "GND") (footprint "")
     )
-    (path "/5873cb1d-2980-4d04-84de-c428523b74e7/9d6541bd-89ef-4879-804a-48e3c42ca566"
+    (path "/1e5d0253-acc2-4f0d-86a2-9343225c71a7/9d250b91-136a-47fa-a162-935e32c2812f"
       (reference "#PWR0109") (unit 1) (value "GND") (footprint "")
     )
@@
       (reference "C6") (unit 1) (value "TBD") (footprint "Capacitor_SMD:C_0603_1608Metric")
     )
+    (path "/1e5d0253-acc2-4f0d-86a2-9343225c71a7/12979e26-efd0-4e90-9283-e94ed728f142"
+      (reference "C7") (unit 1) (value "0.1uF") (footprint "Capacitor_SMD:C_0603_1608Metric")
+    )
+    (path "/1e5d0253-acc2-4f0d-86a2-9343225c71a7/2fa4a35f-e1e3-4656-8c62-24ec47434db9"
+      (reference "C8") (unit 1) (value "10uF") (footprint "Capacitor_SMD:C_0603_1608Metric")
+    )
     (path "/5873cb1d-2980-4d04-84de-c428523b74e7/f18d7b7b-e771-4659-b7d2-4766cb7b211d"
       (reference "C9") (unit 1) (value ".1uF") (footprint "Capacitor_SMD:C_0603_1608Metric")
@@
       (reference "C12") (unit 1) (value "7pF") (footprint "Capacitor_SMD:C_0603_1608Metric")
     )
+    (path "/1e5d0253-acc2-4f0d-86a2-9343225c71a7/efa0f77d-41bc-4b01-a0a8-aedd88523cdc"
+      (reference "C13") (unit 1) (value "0.1uF") (footprint "Capacitor_SMD:C_0603_1608Metric")
+    )
+    (path "/1e5d0253-acc2-4f0d-86a2-9343225c71a7/2434846a-0bdd-4519-8b7f-28daa1f4fdef"
+      (reference "C14") (unit 1) (value "10uF") (footprint "Capacitor_SMD:C_0603_1608Metric")
+    )
     (path "/5873cb1d-2980-4d04-84de-c428523b74e7/90717e53-b8a8-410e-80a8-6872bbb592cd"
       (reference "D1") (unit 1) (value "DSS13UTR") (footprint "Diode_SMD:D_SOD-123F")
     )
-    (path "/1e5d0253-acc2-4f0d-86a2-9343225c71a7/572c9e75-2154-43e6-b982-b5f4a3656d77"
-      (reference "H1") (unit 1) (value "MountingHole") (footprint "MountingHole:MountingHole_2.5mm")
-    )
     (path "/5873cb1d-2980-4d04-84de-c428523b74e7/a758c4bb-94d9-4684-b84b-05442dca5332"
-      (reference "J1") (unit 1) (value "SMA") (footprint "Connector_Coaxial:SMA_Amphenol_901-143_Horizontal")
+      (reference "J1") (unit 1) (value "SMA") (footprint "Connector_Coaxial:SMA_Amphenol_132134_Vertical")
     )
     (path "/5873cb1d-2980-4d04-84de-c428523b74e7/7f2b987d-c54d-48dc-baee-31991a9bc8e8"
       (reference "J2") (unit 1) (value "Molex 0480370001") (footprint "JoesFootprints:Molex_0480370001")
     )
-    (path "/1e5d0253-acc2-4f0d-86a2-9343225c71a7/fdae2716-24d7-4b8d-b7f7-a6b29d466701"
-      (reference "J4") (unit 1) (value "RST") (footprint "Connector_PinHeader_2.54mm:PinHeader_1x02_P2.54mm_Vertical")
-    )
     (path "/5873cb1d-2980-4d04-84de-c428523b74e7/43528de2-bdae-4302-9d4a-272f7ba16a79"
-      (reference "L1") (unit 1) (value "L") (footprint "")
+      (reference "L1") (unit 1) (value "TBD") (footprint "Inductor_SMD:L_0805_2012Metric_Pad1.15x1.40mm_HandSolder")
     )
     (path "/1e5d0253-acc2-4f0d-86a2-9343225c71a7/9a1c7ab1-dc06-4fa0-8127-248c75dab7d9"
@@
       (reference "R3") (unit 1) (value "10k") (footprint "Resistor_SMD:R_0805_2012Metric")
     )
-    (path "/5873cb1d-2980-4d04-84de-c428523b74e7/b2eaf24f-bc7d-48ea-aa0c-4eeba5154b9b"
-      (reference "R7") (unit 1) (value "22") (footprint "Resistor_SMD:R_0805_2012Metric")
+    (path "/5873cb1d-2980-4d04-84de-c428523b74e7/c275d594-0005-4b2c-8157-fcf624c5ebe6"
+      (reference "R4") (unit 1) (value "22") (footprint "Resistor_SMD:R_0805_2012Metric")
     )
-    (path "/5873cb1d-2980-4d04-84de-c428523b74e7/c6d48923-4fe2-4bf5-8474-58c84d705d1d"
-      (reference "R8") (unit 1) (value "22") (footprint "Resistor_SMD:R_0805_2012Metric")
+    (path "/5873cb1d-2980-4d04-84de-c428523b74e7/b6ee8426-c15d-44e0-b16b-218fd6a536b6"
+      (reference "R5") (unit 1) (value "22") (footprint "Resistor_SMD:R_0805_2012Metric")
+    )
+    (path "/1e5d0253-acc2-4f0d-86a2-9343225c71a7/c43eb677-07db-4d19-a565-799396c3e905"
+      (reference "SW1") (unit 1) (value "434133025816") (footprint "Button_Switch_SMD:SW_Push_1P1T_NO_Vertical_Wuerth_434133025816")
     )
     (path "/1e5d0253-acc2-4f0d-86a2-9343225c71a7/b97ff70e-3997-4b11-bc73-1102f98616a3"
